Commit message: Fixed portability issue

File: src/Panda/panda.urdf (robot description, URDF)
Before this commit: robot panda, 12 links, 11 joints
Links:
- link panda_hand: geometry collision mesh filename=package://panda_urdf_modifications/meshes/collision/hand.stl; visual mesh filename=package://panda_urdf_modifications/meshes/visual/hand.dae
- link panda_leftfinger: geometry collision mesh filename=package://panda_urdf_modifications/meshes/collision/finger.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; visual mesh filename=package://panda_urdf_modifications/meshes/visual/finger.dae
- link panda_link0: geometry collision mesh filename=package://panda_urdf_modifications/meshes/collision/link0.s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; visual mesh filename=package://panda_urdf_modifications/meshes/visual/link0.dae
- link panda_link1: geometry collision mesh filename=package://panda_urdf_modifications/meshes/collision/link1.s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; visual mesh filename=package://panda_urdf_modifications/meshes/visual/link1.dae
- link panda_link2: geometry collision mesh filename=package://panda_urdf_modifications/meshes/collision/link2.s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; visual mesh filename=package://panda_urdf_modifications/meshes/visual/link2.dae
- link panda_link3: geometry collision mesh filename=package://panda_urdf_modifications/meshes/collision/link3.s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; visual mesh filename=package://panda_urdf_modifications/meshes/visual/link3.dae
- link panda_link4: geometry collision mesh filename=package://panda_urdf_modifications/meshes/collision/link4.s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; visual mesh filename=package://panda_urdf_modifications/meshes/visual/link4.dae
- link panda_link5: geometry collision mesh filename=package://panda_urdf_modifications/meshes/collision/link5.s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; visual mesh filename=package://panda_urdf_modifications/meshes/visual/link5.dae
- link panda_link6: geometry collision mesh filename=package://panda_urdf_modifications/meshes/collision/link6.s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; visual mesh filename=package://panda_urdf_modifications/meshes/visual/link6.dae
- link panda_link7: geometry collision mesh filename=package://panda_urdf_modifications/meshes/collision/link7.s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; visual mesh filename=package://panda_urdf_modifications/meshes/visual/link7.dae
- link panda_rightfinger: geometry collision mesh filename=package://panda_urdf_modifications/meshes/collision/finger.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; visual mesh filename=package://panda_urdf_modifications/meshes/visual/finger.dae

File: src/custom_config/config/panda.urdf.xacro (robot description, xacro)
@@ -2,7 +2,7 @@
 <robot xmlns:xacro="http://www.ros.org/wiki/xacro" name="panda">
     <xacro:arg name="initial_positions_file" default="initial_positions.yaml" />
-    <!-- Import panda urdf file -->
-    <xacro:include filename="/home/nick/panda_dof_ws/src/Panda/panda.urdf" />
-    <!-- Import control_xacro -->
+    <!-- Including another xacro from a different package: -->
+    <xacro:include filename="package://panda_urdf_modifications/urdf/panda_7dof.urdf.xacro" />
+    <!-- Including another xacro from the same folder (relative): -->
     <xacro:include filename="panda.ros2_control.xacro" />
     <xacro:panda_ros2_control name="FakeSystem" initial_positions_file="$(arg initial_positions_file)"/>

File: src/panda_0dof_moveit_config/urdf/panda.urdf (robot description, URDF)
Before this commit: robot panda, 12 links, 11 joints
Links:
- link panda_hand: geometry collision mesh filename=package://panda_urdf_modifications/meshes/collision/hand.stl; visual mesh filename=package://panda_urdf_modifications/meshes/visual/hand.dae
- link panda_leftfinger: geometry collision mesh filename=package://panda_urdf_modifications/meshes/collision/finger.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; visual mesh filename=package://panda_urdf_modifications/meshes/visual/finger.dae
- link panda_link0: geometry collision mesh filename=package://panda_urdf_modifications/meshes/collision/link0.s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; visual mesh filename=package://panda_urdf_modifications/meshes/visual/link0.dae
- link panda_link1: geometry collision mesh filename=package://panda_urdf_modifications/meshes/collision/link1.s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; visual mesh filename=package://panda_urdf_modifications/meshes/visual/link1.dae
- link panda_link2: geometry collision mesh filename=package://panda_urdf_modifications/meshes/collision/link2.s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; visual mesh filename=package://panda_urdf_modifications/meshes/visual/link2.dae
- link panda_link3: geometry collision mesh filename=package://panda_urdf_modifications/meshes/collision/link3.s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; visual mesh filename=package://panda_urdf_modifications/meshes/visual/link3.dae
- link panda_link4: geometry collision mesh filename=package://panda_urdf_modifications/meshes/collision/link4.s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; visual mesh filename=package://panda_urdf_modifications/meshes/visual/link4.dae
- link panda_link5: geometry collision mesh filename=package://panda_urdf_modifications/meshes/collision/link5.s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; visual mesh filename=package://panda_urdf_modifications/meshes/visual/link5.dae
- link panda_link6: geometry collision mesh filename=package://panda_urdf_modifications/meshes/collision/link6.s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; visual mesh filename=package://panda_urdf_modifications/meshes/visual/link6.dae
- link panda_link7: geometry collision mesh filename=package://panda_urdf_modifications/meshes/collision/link7.s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; visual mesh filename=package://panda_urdf_modifications/meshes/visual/link7.dae
- link panda_rightfinger: geometry collision mesh filename=package://panda_urdf_modifications/meshes/collision/finger.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; visual mesh filename=package://panda_urdf_modifications/meshes/visual/finger.dae

File: src/panda_4dof_moveit_config/urdf/panda.urdf (robot description, URDF)
Before this commit: robot panda, 12 links, 11 joints
Links:
- link panda_hand: geometry collision mesh filename=package://panda_urdf_modifications/meshes/collision/hand.stl; visual mesh filename=package://panda_urdf_modifications/meshes/visual/hand.dae
- link panda_leftfinger: geometry collision mesh filename=package://panda_urdf_modifications/meshes/collision/finger.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; visual mesh filename=package://panda_urdf_modifications/meshes/visual/finger.dae
- link panda_link0: geometry collision mesh filename=package://panda_urdf_modifications/meshes/collision/link0.s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; visual mesh filename=package://panda_urdf_modifications/meshes/visual/link0.dae
- link panda_link1: geometry collision mesh filename=package://panda_urdf_modifications/meshes/collision/link1.s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; visual mesh filename=package://panda_urdf_modifications/meshes/visual/link1.dae
- link panda_link2: geometry collision mesh filename=package://panda_urdf_modifications/meshes/collision/link2.s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; visual mesh filename=package://panda_urdf_modifications/meshes/visual/link2.dae
- link panda_link3: geometry collision mesh filename=package://panda_urdf_modifications/meshes/collision/link3.s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; visual mesh filename=package://panda_urdf_modifications/meshes/visual/link3.dae
- link panda_link4: geometry collision mesh filename=package://panda_urdf_modifications/meshes/collision/link4.s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; visual mesh filename=package://panda_urdf_modifications/meshes/visual/link4.dae
- link panda_link5: geometry collision mesh filename=package://panda_urdf_modifications/meshes/collision/link5.s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; visual mesh filename=package://panda_urdf_modifications/meshes/visual/link5.dae
- link panda_link6: geometry collision mesh filename=package://panda_urdf_modifications/meshes/collision/link6.s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; visual mesh filename=package://panda_urdf_modifications/meshes/visual/link6.dae
- link panda_link7: geometry collision mesh filename=package://panda_urdf_modifications/meshes/collision/link7.s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; visual mesh filename=package://panda_urdf_modifications/meshes/visual/link7.dae
- link panda_rightfinger: geometry collision mesh filename=package://panda_urdf_modifications/meshes/collision/finger.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; visual mesh filename=package://panda_urdf_modifications/meshes/visual/finger.dae

File: src/panda_5dof_moveit_config/urdf/panda.urdf (robot description, URDF)
Before this commit: robot panda, 12 links, 11 joints
Links:
- link panda_hand: geometry collision mesh filename=package://panda_urdf_modifications/meshes/collision/hand.stl; visual mesh filename=package://panda_urdf_modifications/meshes/visual/hand.dae
- link panda_leftfinger: geometry collision mesh filename=package://panda_urdf_modifications/meshes/collision/finger.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; visual mesh filename=package://panda_urdf_modifications/meshes/visual/finger.dae
- link panda_link0: geometry collision mesh filename=package://panda_urdf_modifications/meshes/collision/link0.s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; visual mesh filename=package://panda_urdf_modifications/meshes/visual/link0.dae
- link panda_link1: geometry collision mesh filename=package://panda_urdf_modifications/meshes/collision/link1.s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; visual mesh filename=package://panda_urdf_modifications/meshes/visual/link1.dae
- link panda_link2: geometry collision mesh filename=package://panda_urdf_modifications/meshes/collision/link2.s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; visual mesh filename=package://panda_urdf_modifications/meshes/visual/link2.dae
- link panda_link3: geometry collision mesh filename=package://panda_urdf_modifications/meshes/collision/link3.s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; visual mesh filename=package://panda_urdf_modifications/meshes/visual/link3.dae
- link panda_link4: geometry collision mesh filename=package://panda_urdf_modifications/meshes/collision/link4.s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; visual mesh filename=package://panda_urdf_modifications/meshes/visual/link4.dae
- link panda_link5: geometry collision mesh filename=package://panda_urdf_modifications/meshes/collision/link5.s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; visual mesh filename=package://panda_urdf_modifications/meshes/visual/link5.dae
- link panda_link6: geometry collision mesh filename=package://panda_urdf_modifications/meshes/collision/link6.s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; visual mesh filename=package://panda_urdf_modifications/meshes/visual/link6.dae
- link panda_link7: geometry collision mesh filename=package://panda_urdf_modifications/meshes/collision/link7.s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; visual mesh filename=package://panda_urdf_modifications/meshes/visual/link7.dae
- link panda_rightfinger: geometry collision mesh filename=package://panda_urdf_modifications/meshes/collision/finger.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; visual mesh filename=package://panda_urdf_modifications/meshes/visual/finger.dae

File: src/panda_6dof_moveit_config/urdf/panda.urdf (robot description, URDF)
Before this commit: robot panda, 12 links, 11 joints
Links:
- link panda_hand: geometry collision mesh filename=package://panda_urdf_modifications/meshes/collision/hand.stl; visual mesh filename=package://panda_urdf_modifications/meshes/visual/hand.dae
- link panda_leftfinger: geometry collision mesh filename=package://panda_urdf_modifications/meshes/collision/finger.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; visual mesh filename=package://panda_urdf_modifications/meshes/visual/finger.dae
- link panda_link0: geometry collision mesh filename=package://panda_urdf_modifications/meshes/collision/link0.s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; visual mesh filename=package://panda_urdf_modifications/meshes/visual/link0.dae
- link panda_link1: geometry collision mesh filename=package://panda_urdf_modifications/meshes/collision/link1.s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; visual mesh filename=package://panda_urdf_modifications/meshes/visual/link1.dae
- link panda_link2: geometry collision mesh filename=package://panda_urdf_modifications/meshes/collision/link2.s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; visual mesh filename=package://panda_urdf_modifications/meshes/visual/link2.dae
- link panda_link3: geometry collision mesh filename=package://panda_urdf_modifications/meshes/collision/link3.s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; visual mesh filename=package://panda_urdf_modifications/meshes/visual/link3.dae
- link panda_link4: geometry collision mesh filename=package://panda_urdf_modifications/meshes/collision/link4.s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; visual mesh filename=package://panda_urdf_modifications/meshes/visual/link4.dae
- link panda_link5: geometry collision mesh filename=package://panda_urdf_modifications/meshes/collision/link5.s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; visual mesh filename=package://panda_urdf_modifications/meshes/visual/link5.dae
- link panda_link6: geometry collision mesh filename=package://panda_urdf_modifications/meshes/collision/link6.s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; visual mesh filename=package://panda_urdf_modifications/meshes/visual/link6.dae
- link panda_link7: geometry collision mesh filename=package://panda_urdf_modifications/meshes/collision/link7.s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; visual mesh filename=package://panda_urdf_modifications/meshes/visual/link7.dae
- link panda_rightfinger: geometry collision mesh filename=package://panda_urdf_modifications/meshes/collision/finger.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; visual mesh filename=package://panda_urdf_modifications/meshes/visual/finger.dae

File: src/panda_7dof_moveit_config/config/panda.urdf.xacro (robot description, xacro)
@@ -4,5 +4,5 @@
     <xacro:arg name="ros2_control_hardware_type" default="mock_components" />
     <!-- Import panda urdf file -->
-    <xacro:include filename="$(find_pkg panda_urdf_modifications)/urdf/panda_7dof.urdf.xacro"/>
+    <xacro:include filename="$(find panda_urdf_modifications)/urdf/panda_7dof.urdf.xacro"/>
     <!-- Import panda ros2_control description -->
     <xacro:include filename="panda.ros2_control.xacro" />
