Commit message: All DOFs Working

File: src/panda_1dof_moveit_config/urdf/panda.urdf (robot description, URDF)
Before this commit: robot panda, 12 links, 11 joints
Links:
- link panda_hand: geometry collision mesh filename=package://panda_urdf_modifications/meshes/collision/hand.obj; visual mesh filename=package://panda_urdf_modifications/meshes/visual/hand.dae
- link panda_leftfinger: geometry collision mesh filename=package://panda_urdf_modifications/meshes/collision/finger.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; visual mesh filename=package://panda_urdf_modifications/meshes/visual/finger.dae
- link panda_link0: geometry collision mesh filename=package://panda_urdf_modifications/meshes/collision/link0.o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; visual mesh filename=package://panda_urdf_modifications/meshes/visual/link0.dae
- link panda_link1: geometry collision mesh filename=package://panda_urdf_modifications/meshes/collision/link1.o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; visual mesh filename=package://panda_urdf_modifications/meshes/visual/link1.dae
- link panda_link2: geometry collision mesh filename=package://panda_urdf_modifications/meshes/collision/link2.o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; visual mesh filename=package://panda_urdf_modifications/meshes/visual/link2.dae
- link panda_link3: geometry collision mesh filename=package://panda_urdf_modifications/meshes/collision/link3.o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; visual mesh filename=package://panda_urdf_modifications/meshes/visual/link3.dae
- link panda_link4: geometry collision mesh filename=package://panda_urdf_modifications/meshes/collision/link4.o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; visual mesh filename=package://panda_urdf_modifications/meshes/visual/link4.dae
- link panda_link5: geometry collision mesh filename=package://panda_urdf_modifications/meshes/collision/link5.o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; visual mesh filename=package://panda_urdf_modifications/meshes/visual/link5.dae
- link panda_link6: geometry collision mesh filename=package://panda_urdf_modifications/meshes/collision/link6.o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; visual mesh filename=package://panda_urdf_modifications/meshes/visual/link6.dae
- link panda_link7: geometry collision mesh filename=package://panda_urdf_modifications/meshes/collision/link7.o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; visual mesh filename=package://panda_urdf_modifications/meshes/visual/link7.dae
- link panda_rightfinger: geometry collision mesh filename=package://panda_urdf_modifications/meshes/collision/finger.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; visual mesh filename=package://panda_urdf_modifications/meshes/visual/finger.dae

File: src/panda_2dof_moveit_config/urdf/panda.urdf (robot description, URDF)
Before this commit: robot panda, 12 links, 11 joints
Links:
- link panda_hand: geometry collision mesh filename=package://panda_urdf_modifications/meshes/collision/hand.obj; visual mesh filename=package://panda_urdf_modifications/meshes/visual/hand.dae
- link panda_leftfinger: geometry collision mesh filename=package://panda_urdf_modifications/meshes/collision/finger.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; visual mesh filename=package://panda_urdf_modifications/meshes/visual/finger.dae
- link panda_link0: geometry collision mesh filename=package://panda_urdf_modifications/meshes/collision/link0.o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; visual mesh filename=package://panda_urdf_modifications/meshes/visual/link0.dae
- link panda_link1: geometry collision mesh filename=package://panda_urdf_modifications/meshes/collision/link1.o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; visual mesh filename=package://panda_urdf_modifications/meshes/visual/link1.dae
- link panda_link2: geometry collision mesh filename=package://panda_urdf_modifications/meshes/collision/link2.o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; visual mesh filename=package://panda_urdf_modifications/meshes/visual/link2.dae
- link panda_link3: geometry collision mesh filename=package://panda_urdf_modifications/meshes/collision/link3.o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; visual mesh filename=package://panda_urdf_modifications/meshes/visual/link3.dae
- link panda_link4: geometry collision mesh filename=package://panda_urdf_modifications/meshes/collision/link4.o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; visual mesh filename=package://panda_urdf_modifications/meshes/visual/link4.dae
- link panda_link5: geometry collision mesh filename=package://panda_urdf_modifications/meshes/collision/link5.o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; visual mesh filename=package://panda_urdf_modifications/meshes/visual/link5.dae
- link panda_link6: geometry collision mesh filename=package://panda_urdf_modifications/meshes/collision/link6.o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; visual mesh filename=package://panda_urdf_modifications/meshes/visual/link6.dae
- link panda_link7: geometry collision mesh filename=package://panda_urdf_modifications/meshes/collision/link7.o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; visual mesh filename=package://panda_urdf_modifications/meshes/visual/link7.dae
- link panda_rightfinger: geometry collision mesh filename=package://panda_urdf_modifications/meshes/collision/finger.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; visual mesh filename=package://panda_urdf_modifications/meshes/visual/finger.dae

File: src/panda_3dof_moveit_config/urdf/panda.urdf (robot description, URDF)
Before this commit: robot panda, 12 links, 11 joints
Links:
- link panda_hand: geometry collision mesh filename=package://panda_urdf_modifications/meshes/collision/hand.obj; visual mesh filename=package://panda_urdf_modifications/meshes/visual/hand.dae
- link panda_leftfinger: geometry collision mesh filename=package://panda_urdf_modifications/meshes/collision/finger.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; visual mesh filename=package://panda_urdf_modifications/meshes/visual/finger.dae
- link panda_link0: geometry collision mesh filename=package://panda_urdf_modifications/meshes/collision/link0.o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; visual mesh filename=package://panda_urdf_modifications/meshes/visual/link0.dae
- link panda_link1: geometry collision mesh filename=package://panda_urdf_modifications/meshes/collision/link1.o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; visual mesh filename=package://panda_urdf_modifications/meshes/visual/link1.dae
- link panda_link2: geometry collision mesh filename=package://panda_urdf_modifications/meshes/collision/link2.o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; visual mesh filename=package://panda_urdf_modifications/meshes/visual/link2.dae
- link panda_link3: geometry collision mesh filename=package://panda_urdf_modifications/meshes/collision/link3.o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; visual mesh filename=package://panda_urdf_modifications/meshes/visual/link3.dae
- link panda_link4: geometry collision mesh filename=package://panda_urdf_modifications/meshes/collision/link4.o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; visual mesh filename=package://panda_urdf_modifications/meshes/visual/link4.dae
- link panda_link5: geometry collision mesh filename=package://panda_urdf_modifications/meshes/collision/link5.o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; visual mesh filename=package://panda_urdf_modifications/meshes/visual/link5.dae
- link panda_link6: geometry collision mesh filename=package://panda_urdf_modifications/meshes/collision/link6.o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; visual mesh filename=package://panda_urdf_modifications/meshes/visual/link6.dae
- link panda_link7: geometry collision mesh filename=package://panda_urdf_modifications/meshes/collision/link7.o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; visual mesh filename=package://panda_urdf_modifications/meshes/visual/link7.dae
- link panda_rightfinger: geometry collision mesh filename=package://panda_urdf_modifications/meshes/collision/finger.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; visual mesh filename=package://panda_urdf_modifications/meshes/visual/finger.dae
